File: ErdferkelEStopPCB/ErdferkelEStopPCB/ErdferkelEStopPCB.kicad_pcb (KiCad board)
At the start: 2 copper layers, 60 x 80 mm, 9 parts, among them J1 Screw_Terminal_01x02, J2 Conn_01x10_Pin, J3 Conn_01x10_Pin, J4 Conn_01x19_Pin, J5 Conn_01x19_Pin, J6 Screw_Terminal_01x02, Q1 S8050

Commit message: EStop PCB: Replace S8050 with SS8050
We want to have all SMD components on this to reduce size.
Parts:
- removed Q1: S8050, Package_TO_SOT_THT:TO-92_Inline
- added Q2: SS8050, Package_TO_SOT_SMD:SOT-23, F.Cu at (135.5, 98.0)
Routing:
- net Net-(Q2-B): track 10.8 -> 9.12 mm
- net Net-(J1-Pin_2): track 13.1 -> 11.6 mm
